File: pcb/aW_2/aW_2.kicad_pcb (KiCad board)
At the start: 2 copper layers, 112 parts, among them J1 USB4110-GF-A, J2 USB4110-GF-A, J3 USB4110-GF-A, J4 Conn_ARM_JTAG_SWD_10, K1 KEYSW, K10 KEYSW, K11 KEYSW, K12 KEYSW, K13 KEYSW, K14 KEYSW, K15 KEYSW, K16 KEYSW, K17 KEYSW, K18 KEYSW, K19 KEYSW, K2 KEYSW, K20 KEYSW, K21 KEYSW, K22 KEYSW, K23 KEYSW, K24 KEYSW, K25 KEYSW, K26 KEYSW, K27 KEYSW, K28 KEYSW, K29 KEYSW, K3 KEYSW, K30 KEYSW, K31 KEYSW, K32 KEYSW, K33 KEYSW, K4 KEYSW, K5 KEYSW, K6 KEYSW, K7 KEYSW, K8 KEYSW, K9 KEYSW, Q1 Q_PMOS_SDG, SW1 BTN1, SW2 BTN2, U1 AP2112K-3.3TRG1, U2 MCP23017T-E_SS, U3 MCP73831-2-OT, U4 FT231XS-R, U5 BL652-SA-01-T_R, Y1 32.768

Commit message: (Almost) finished pcb, few GND connections missing
Parts:
- J4: moved to B.Cu
- moved R2 103.1 mm to (197.8, 162.8)
- moved D1 98.6 mm to (194.8, 162.8)
- moved Q1 93.4 mm to (194.8, 159.3), turned to 270 degrees
- moved R3 92.2 mm to (188.9, 162.8), turned to 90 degrees
- moved C3 89.9 mm to (191.3, 162.8), turned to 270 degrees
- moved D2 86.0 mm to (154.0, 156.3), turned to 90 degrees
- moved U1 82.8 mm to (188.9, 159.2), turned to 180 degrees
- moved C2 80.5 mm to (187.1, 162.8)
- moved SW2 79.9 mm to (161.1, 156.9), turned to 270 degrees
- moved C4 73.8 mm to (201.3, 162.8), turned to 270 degrees
- moved D36 73.5 mm to (151.6, 156.3), turned to 270 degrees
- moved C5 66.2 mm to (204.9, 162.8), turned to 270 degrees
- moved BT1 64.9 mm to (233.9, 160.5), turned to 270 degrees
- moved SW1 64.3 mm to (164.6, 156.9), turned to 270 degrees
- moved JP1 63.6 mm to (109.0, 162.8), turned to 270 degrees
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Routing:
- net /sda_right: track 0.00 -> 346.3 mm, vias 0 -> 2
- net /scl_right: track 0.00 -> 343.6 mm, vias 0 -> 2
- net +3V3: track 148.6 -> 274.7 mm, vias 4 -> 10
- net VBUS: track 0.00 -> 102.5 mm, vias 0 -> 5
- net GND: track 0.00 -> 62.6 mm, vias 0 -> 19
- net +BATT: track 0.00 -> 54.1 mm
- net Net-(D2-Pad1): track 0.00 -> 53.7 mm, vias 0 -> 2
- net /reset: track 0.00 -> 49.4 mm, vias 0 -> 2
- net /btn2: track 0.00 -> 48.9 mm, vias 0 -> 2
- net Net-(C6-Pad1): track 0.00 -> 32.5 mm, vias 0 -> 2
- net /main_usb_dp: track 0.00 -> 29.5 mm
- net /main_usb_dn: track 0.00 -> 29.5 mm
- net /led1: track 0.00 -> 28.9 mm, vias 0 -> 2
- net Net-(JP1-Pad2): track 0.00 -> 16.0 mm, vias 0 -> 2
- net Net-(R8-Pad1): track 0.00 -> 16.0 mm, vias 0 -> 2
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- added copper zone on B.Cu, net GND
- added copper zone on F.Cu, net GND
Other:
- board outline added: 143.3 x 113.1 mm

Commit message: Traces and pours finished
Parts:
- J4: moved to F.Cu
- moved J4 1.18 mm to (129.7, 156.3), turned to 90 degrees
- moved SW1 0.59 mm to (165.2, 156.9)
- moved C11 0.59 mm to (132.0, 161.1)
Connections:
- C1 pad 1: +3V3 -> VDC
- J1 pad A4/B9: +3V3 -> VDC
- J1 pad B4/A9: +3V3 -> VDC
- R1 pad 1: +3V3 -> VDC
- U2 pad 9: +3V3 -> VDC
Routing:
- net VDC: track 0.00 -> 143.1 mm, vias 0 -> 4
- net +3V3: track 274.7 -> 206.2 mm, vias 10 -> 6
- net GND: track 62.6 -> 92.4 mm, vias 19 -> 28
- net /swo: track 9.49 -> 20.8 mm
- net /swdclk: track 7.12 -> 12.2 mm, vias 0 -> 2
- net /uart_rx: track 15.5 -> 18.5 mm
- net /swdio: track 5.81 -> 8.30 mm
- net /uart_tx: track 11.1 -> 12.0 mm
- net /sda_left: track 116.2 -> 115.4 mm
- net /scl_left: track 117.4 -> 116.6 mm
- net /btn2: track 48.9 -> 48.0 mm
- net /reset: track 49.4 -> 50.2 mm, vias 2 -> 3

Commit message: Fixed silk screen and fab layers
Parts:
- D1: value D_Schottky -> Schottky
- J4: value Conn_ARM_JTAG_SWD_10 -> JTAG_SWD; footprint Connector_PinHeader_1.27mm:PinHeader_2x05_P1.27mm_Horizontal -> Connector_PinHeader_1.27mm:PinHeader_2x05_P1.27mm_Vertical
- JP1: value SolderJumper_3_Open -> Jumper_3_Open
- Q1: value Q_PMOS_SDG -> P_SDG
- U1: value AP2112K-3.3TRG1 -> AP2112K-3.3
- U3: value MCP73831-2-OT -> MCP73831
Routing:
- net GND: track 92.4 -> 93.1 mm

Commit message: Added gerbers, license information, updated connector information
Parts:
- added S1: JS202011JAQN, snap-eda:JS202011JAQN, F.Cu at (165.8, 33.2)
- D1: value Schottky -> D_Schottky
- J4: value JTAG_SWD -> Conn_ARM_JTAG_SWD_10
- JP1: value Jumper_3_Open -> SolderJumper_3_Open
- Q1: value P_SDG -> Q_PMOS_SDG
- U1: value AP2112K-3.3 -> AP2112K-3.3TRG1
- U3: value MCP73831 -> MCP73831-2-OT
- moved J3 127.6 mm to (142.1, 35.5)
- moved R4 127.6 mm to (147.4, 38.5)
- moved R5 127.6 mm to (136.8, 38.5)
- moved BT1 125.3 mm to (198.4, 40.3)
- moved C1 125.3 mm to (103.0, 43.2)
- moved C7 125.3 mm to (115.5, 43.2)
- moved D16 125.3 mm to (198.4, 82.3)
- moved K10 125.3 mm to (127.9, 77.5)
- moved K11 125.3 mm to (146.9, 77.5)
- moved K12 125.3 mm to (165.8, 77.5)
- moved K13 125.3 mm to (184.8, 77.5)
- moved K14 125.3 mm to (203.7, 82.2)
- moved K8 125.3 mm to (85.3, 77.5)
- moved K9 125.3 mm to (109.0, 77.5)
- moved R8 125.3 mm to (120.2, 43.2)
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Connections:
- C2 pad 1: +3V3 -> Net-(C2-Pad1)
- U1 pad 5: +3V3 -> Net-(C2-Pad1)
Routing:
- net Net-(C2-Pad1): track 0.00 -> 35.9 mm
- net +BATT: track 54.1 -> 59.2 mm
- net GND: track 93.1 -> 98.0 mm, vias 28 -> 27
- net +3V3: track 206.2 -> 209.9 mm, vias 6 -> 8
- net Net-(D2-Pad1): track 53.7 -> 56.4 mm
- net /main_usb_dp: track 29.5 -> 32.1 mm
- net /main_usb_dn: track 29.5 -> 31.9 mm
- net /sda_left: track 115.4 -> 117.5 mm
- net /scl_left: track 116.6 -> 118.7 mm
- net VDC: track 143.1 -> 145.3 mm
- net /scl_right: track 343.6 -> 342.0 mm
- net /sda_right: track 346.3 -> 344.8 mm
- net VBUS: track 102.5 -> 103.3 mm
Other:
- board size 143.3 x 113.1 mm -> 145.1 x 114.9 mm
